Commit message: task space works (maybe)

File: catkin_ws/src/giraffe_description/urdf/generated_urdf/giraffe.urdf (robot description, URDF)
Before this commit: robot giraffe_robot, 7 links, 6 joints
Links:
- link base_link: mass 2.0 -> 5.0
- link ee_link: mass 0.05 -> 0.3; geometry collision sphere radius=0.03; visual box size=0.03 0.03 0.03
- link link1: mass 0.3 -> 1.0
- link link2: mass 0.7 -> 2.0
- link link3: mass 0.3 -> 1.5; geometry collision box size=0.1 0.1 0.1; visual box size=0.1 0.1 0.1
- link link4: mass 0.1 -> 0.5
Joints:
- joint joint1: origin xyz=0 0 0 rpy=0 3.141592653589793 0 -> xyz=0 0 0.025 rpy=0 0 0
- joint joint2: limit lower=-3.141592653589793 upper=0 effort=100 velocity=1 -> lower=-2.0943951023931953 upper=0 effort=100 velocity=1
- joint joint3: limit lower=0 upper=6.5 effort=10000 velocity=0.5 -> lower=0 upper=3.0 effort=10000 velocity=0.5

File: catkin_ws/src/giraffe_description/urdf/giraffe.urdf.xacro (robot description, xacro)
@@ -5,16 +5,16 @@
   <xacro:property name="ceiling_height" value="4.0" />
   <xacro:property name="arm_segment_length" value="0.5" />
-  <xacro:property name="prismatic_max_extension" value="6.5" />
+  <xacro:property name="prismatic_max_extension" value="3.0" />  <!-- Reduced from 6.5m -->
   <xacro:property name="mic_arm_length" value="0.3" />
   <!-- Materials -->
-  <material name="gray"><color rgba="0 0 0 1"/></material>
+  <material name="gray"><color rgba="0.5 0.5 0.5 1"/></material>
   <material name="red"><color rgba="1 0 0 1"/></material>
-  <material name="green"><color rgba="1 1 0 1"/></material>
-  <material name="blue"><color rgba="1 0 0 1"/></material>
+  <material name="green"><color rgba="0 1 0 1"/></material>  <!-- Fixed color -->
+  <material name="blue"><color rgba="0 0 1 1"/></material>   <!-- Fixed color -->
   <material name="yellow"><color rgba="1 1 0 1"/></material>
   <material name="black"><color rgba="0 0 0 1"/></material>
   <material name="white"><color rgba="1 1 1 1"/></material>
   <link name="world"/>
-  <!-- Base -->
+  <!-- Base - Increased mass and corrected inertia -->
   <link name="base_link">
     <visual>
@@ -23,11 +23,11 @@
     </visual>
     <collision>
-      <origin xyz="0 0 0" />
       <geometry><box size="0.2 0.2 0.05"/></geometry>
     </collision>
     <inertial>
-      <mass value="2.0"/>
+      <mass value="5.0"/>  <!-- Increased from 2.0 -->
       <origin xyz="0 0 0"/>
-      <inertia ixx="0.003" ixy="0" ixz="0" iyy="0.003" iyz="0" izz="0.0005"/>
+      <!-- Corrected inertia for box: I = 1/12*m*(y²+z²) -->
+      <inertia ixx="0.00417" ixy="0" ixz="0" iyy="0.00417" iyz="0" izz="0.00833"/>
     </inertial>
   </link>
@@ -37,5 +37,5 @@
     <origin xyz="2.5 6.0 ${ceiling_height}" rpy="0 0 0"/>
   </joint>
-  <!-- Link1: Pan -->
+  <!-- Link1: Pan - Corrected inertia for cylinder -->
   <link name="link1">
     <visual>
@@ -44,11 +44,11 @@
     </visual>
     <collision>
-      <origin xyz="0 0 0"/>
       <geometry><cylinder length="0.1" radius="0.05"/></geometry>
     </collision>
     <inertial>
-      <mass value="0.3"/>
+      <mass value="1.0"/>  <!-- Increased from 0.3 -->
       <origin xyz="0 0 0"/>
-      <inertia ixx="0.0001" ixy="0" ixz="0" iyy="0.0001" iyz="0" izz="0.0001"/>
+      <!-- Ixx = Iyy = 1/12*m*(3*r² + h²), Izz = 1/2*m*r² -->
+      <inertia ixx="0.00046" ixy="0" ixz="0" iyy="0.00046" iyz="0" izz="0.00125"/>
     </inertial>
   </link>
@@ -56,9 +56,10 @@
     <parent link="base_link"/>
     <child link="link1"/>
-    <origin xyz="0 0 0" rpy="0 ${M_PI} 0"/>
+    <origin xyz="0 0 0.025" rpy="0 0 0"/>  <!-- Offset from base -->
     <axis xyz="0 0 1"/>
     <limit lower="-${M_PI}" upper="${M_PI}" effort="100" velocity="1"/>
+    <dynamics damping="0.5"/>  <!-- Added damping -->
   </joint>
-  <!-- Link2: Tilt -->
+  <!-- Link2: Tilt - Corrected inertia and COM -->
   <link name="link2">
     <visual>
@@ -72,7 +73,8 @@
     </collision>
     <inertial>
-      <mass value="0.7"/>
-      <origin xyz="${arm_segment_length/2} 0 0" rpy="0 ${M_PI/2} 0"/>
-      <inertia ixx="0.002" ixy="0" ixz="0" iyy="0.002" iyz="0" izz="0.0005"/>
+      <mass value="2.0"/>  <!-- Increased from 0.7 -->
+      <origin xyz="${arm_segment_length/2} 0 0"/>  <!-- COM at center -->
+      <!-- For cylinder along x: Ixx = 1/2*m*r², Iyy=Izz=1/12*m*(3r²+L²) -->
+      <inertia ixx="0.0009" ixy="0" ixz="0" iyy="0.0417" iyz="0" izz="0.0417"/>
     </inertial>
   </link>
@@ -82,20 +84,20 @@
     <origin xyz="0 0 0" rpy="0 0 0"/>
     <axis xyz="0 1 0"/>
-    <limit lower="-${M_PI}" upper="0" effort="100" velocity="1"/>
+    <limit lower="-${2*M_PI/3}" upper="0" effort="100" velocity="1"/> <!-- Reduced range -->
+    <dynamics damping="0.5"/>  <!-- Added damping -->
   </joint>
-  <!-- Link3: Prismatic -->
+  <!-- Link3: Prismatic - Increased mass and corrected inertia -->
   <link name="link3">
     <visual>
-      <geometry><sphere radius="0.05"/></geometry>
+      <geometry><box size="0.1 0.1 0.1"/></geometry>  <!-- More realistic than sphere -->
       <material name="blue"/>
     </visual>
     <collision>
-      <origin xyz="0 0 0"/>
-      <geometry><sphere radius="0.05"/></geometry>
+      <geometry><box size="0.1 0.1 0.1"/></geometry>
     </collision>
     <inertial>
-      <mass value="0.3"/>
+      <mass value="1.5"/>  <!-- Increased from 0.3 -->
       <origin xyz="0 0 0"/>
-      <inertia ixx="0.0001" ixy="0" ixz="0" iyy="0.0001" iyz="0" izz="0.0001"/>
+      <inertia ixx="0.0025" ixy="0" ixz="0" iyy="0.0025" iyz="0" izz="0.0025"/>
     </inertial>
   </link>
@@ -106,7 +108,7 @@
     <axis xyz="1 0 0"/>
     <limit lower="0" upper="${prismatic_max_extension}" effort="10000" velocity="0.5"/>
-    <dynamics damping="5.0" friction="1.0"/>
+    <dynamics damping="10.0" friction="2.0"/>  <!-- Increased damping -->
   </joint>
-  <!-- Link4: Microphone bar -->
+  <!-- Link4: Microphone bar - Corrected inertia -->
   <link name="link4">
     <visual>
@@ -120,7 +122,8 @@
     </collision>
     <inertial>
-      <mass value="0.1"/>
-      <origin xyz="${mic_arm_length/2} 0 0" rpy="0 ${M_PI/2} 0"/>
-      <inertia ixx="0.00005" ixy="0" ixz="0" iyy="0.00005" iyz="0" izz="0.00002"/>
+      <mass value="0.5"/>  <!-- Increased from 0.1 -->
+      <origin xyz="${mic_arm_length/2} 0 0"/>
+      <!-- For cylinder along x: Ixx = 1/2*m*r², Iyy=Izz=1/12*m*(3r²+L²) -->
+      <inertia ixx="0.000025" ixy="0" ixz="0" iyy="0.00377" iyz="0" izz="0.00377"/>
     </inertial>
   </link>
@@ -131,6 +134,7 @@
     <axis xyz="0 1 0"/>
     <limit lower="-${M_PI/2}" upper="${M_PI/2}" effort="50" velocity="1"/>
+    <dynamics damping="0.3"/>  <!-- Added damping -->
   </joint>
-  <!-- End-effector: microphone -->
+  <!-- End-effector: microphone - Corrected inertia -->
   <link name="ee_link">
     <visual>
@@ -149,11 +153,11 @@
     </visual>
     <collision>
-      <origin xyz="0 0 -0.1" rpy="0 0 0"/>
-      <geometry><cylinder length="0.2" radius="0.015"/></geometry>
+      <geometry><sphere radius="0.03"/></geometry>  <!-- Simplified collision -->
     </collision>
     <inertial>
-      <mass value="0.05"/>
-      <origin xyz="0 0 -0.1" rpy="0 0 0"/>
-      <inertia ixx="0.00001" ixy="0" ixz="0" iyy="0.00001" iyz="0" izz="0.000005"/>
+      <mass value="0.3"/>  <!-- Increased from 0.05 -->
+      <origin xyz="0 0 -0.1"/>
+      <!-- Approximate as point mass: I = m*d² -->
+      <inertia ixx="0.003" ixy="0" ixz="0" iyy="0.003" iyz="0" izz="0.003"/>
     </inertial>
   </link>
@@ -164,4 +168,5 @@
     <axis xyz="0 1 0"/>
     <limit lower="-${M_PI/2}" upper="${M_PI/2}" effort="50" velocity="1"/>
+    <dynamics damping="0.2"/>  <!-- Added damping -->
   </joint>
 </robot>

Commit message: urdf modified

File: catkin_ws/src/giraffe_description/urdf/generated_urdf/giraffe.urdf (robot description, URDF)
Before this commit: robot giraffe_robot, 7 links, 6 joints
Links:
- link ee_link: geometry collision sphere radius=0.03; visual cylinder length=0.2 radius=0.008
- link link3: geometry collision cylinder length=6.5 radius=0.03; visual cylinder length=6.5 radius=0.03
- link link4: geometry collision cylinder length=0.3 radius=0.01; visual cylinder length=0.3 radius=0.025
Joints:
- joint joint3: limit lower=0 upper=3.0 effort=10000 velocity=0.5 -> lower=0 upper=6.5 effort=10000 velocity=0.5
- joint joint4: origin xyz=0.05 0 0 rpy=0 0 0 -> xyz=0 0 0 rpy=0 0 0

File: catkin_ws/src/giraffe_description/urdf/giraffe.urdf.xacro (robot description, xacro)
@@ -5,14 +5,11 @@
   <xacro:property name="ceiling_height" value="4.0" />
   <xacro:property name="arm_segment_length" value="0.5" />
-  <xacro:property name="prismatic_max_extension" value="3.0" />  <!-- Reduced from 6.5m -->
+  <xacro:property name="prismatic_max_extension" value="6.5" />
   <xacro:property name="mic_arm_length" value="0.3" />
   <!-- Materials -->
-  <material name="gray"><color rgba="0.5 0.5 0.5 1"/></material>
-  <material name="red"><color rgba="1 0 0 1"/></material>
-  <material name="green"><color rgba="0 1 0 1"/></material>  <!-- Fixed color -->
-  <material name="blue"><color rgba="0 0 1 1"/></material>   <!-- Fixed color -->
-  <material name="yellow"><color rgba="1 1 0 1"/></material>
   <material name="black"><color rgba="0 0 0 1"/></material>
   <material name="white"><color rgba="1 1 1 1"/></material>
+  <material name="dark grey"><color rgba="0 0 0 0.7"/></material>
+  <material name="light grey"><color rgba="0 0 0 0.5"/></material>
   <link name="world"/>
   <!-- Base - Increased mass and corrected inertia -->
@@ -20,5 +17,5 @@
     <visual>
       <geometry><box size="0.2 0.2 0.05"/></geometry>
-      <material name="gray"/>
+      <material name="white"/>
     </visual>
     <collision>
@@ -41,5 +38,5 @@
     <visual>
       <geometry><cylinder length="0.1" radius="0.05"/></geometry>
-      <material name="red"/>
+      <material name="dark grey"/>
     </visual>
     <collision>
@@ -47,7 +44,6 @@
     </collision>
     <inertial>
-      <mass value="1.0"/>  <!-- Increased from 0.3 -->
+      <mass value="1.0"/>
       <origin xyz="0 0 0"/>
-      <!-- Ixx = Iyy = 1/12*m*(3*r² + h²), Izz = 1/2*m*r² -->
       <inertia ixx="0.00046" ixy="0" ixz="0" iyy="0.00046" iyz="0" izz="0.00125"/>
     </inertial>
@@ -59,5 +55,5 @@
     <axis xyz="0 0 1"/>
     <limit lower="-${M_PI}" upper="${M_PI}" effort="100" velocity="1"/>
-    <dynamics damping="0.5"/>  <!-- Added damping -->
+    <dynamics damping="0.5"/>
   </joint>
   <!-- Link2: Tilt - Corrected inertia and COM -->
@@ -66,5 +62,5 @@
       <geometry><cylinder length="${arm_segment_length}" radius="0.03"/></geometry>
       <origin xyz="${arm_segment_length/2} 0 0" rpy="0 ${M_PI/2} 0"/>
-      <material name="green"/>
+      <material name="dark grey"/>
     </visual>
     <collision>
@@ -88,16 +84,18 @@
   </joint>
   <!-- Link3: Prismatic - Increased mass and corrected inertia -->
-  <link name="link3">
+<link name="link3">
     <visual>
-      <geometry><box size="0.1 0.1 0.1"/></geometry>  <!-- More realistic than sphere -->
-      <material name="blue"/>
+      <geometry><cylinder length="${prismatic_max_extension}" radius="0.03"/></geometry>
+      <origin xyz="-${prismatic_max_extension / 2.0} 0 0" rpy="0 ${M_PI/2} 0"/>
+      <material name="dark grey"/>
     </visual>
     <collision>
-      <geometry><box size="0.1 0.1 0.1"/></geometry>
+      <geometry><cylinder length="${prismatic_max_extension}" radius="0.03"/></geometry>
+      <origin xyz="-${prismatic_max_extension / 2.0} 0 0" rpy="0 ${M_PI/2} 0"/>
     </collision>
     <inertial>
-      <mass value="1.5"/>  <!-- Increased from 0.3 -->
-      <origin xyz="0 0 0"/>
-      <inertia ixx="0.0025" ixy="0" ixz="0" iyy="0.0025" iyz="0" izz="0.0025"/>
+      <mass value="1.5"/>
+      <origin xyz="-${prismatic_max_extension / 2.0} 0 0" rpy="0 0 0"/>
+      <inertia ixx="0.0004" ixy="0" ixz="0" iyy="1.1252" iyz="0" izz="1.1252"/>
     </inertial>
   </link>
@@ -113,7 +111,7 @@
   <link name="link4">
     <visual>
-      <geometry><cylinder length="${mic_arm_length}" radius="0.01"/></geometry>
+      <geometry><cylinder length="${mic_arm_length}" radius="0.025"/></geometry>
       <origin xyz="${mic_arm_length/2} 0 0" rpy="0 ${M_PI/2} 0"/>
-      <material name="yellow"/>
+      <material name="light grey"/>
     </visual>
     <collision>
@@ -128,16 +126,16 @@
     </inertial>
   </link>
-  <joint name="joint4" type="revolute">
+<joint name="joint4" type="revolute">
     <parent link="link3"/>
     <child link="link4"/>
-    <origin xyz="0.05 0 0" rpy="0 0 0"/>
+    <origin xyz="0 0 0" rpy="0 0 0"/>
     <axis xyz="0 1 0"/>
     <limit lower="-${M_PI/2}" upper="${M_PI/2}" effort="50" velocity="1"/>
-    <dynamics damping="0.3"/>  <!-- Added damping -->
+    <dynamics damping="0.3"/>
   </joint>
   <!-- End-effector: microphone - Corrected inertia -->
   <link name="ee_link">
     <visual>
-      <geometry><box size="0.03 0.03 0.03"/></geometry>
+      <geometry><sphere radius="0.025"/></geometry>
       <material name="black"/>
     </visual>
@@ -150,13 +148,12 @@
       <geometry><sphere radius="0.015"/></geometry>
       <origin xyz="0 0 -0.2" rpy="0 0 0"/>
-      <material name="red"/>
+      <material name="black"/>
     </visual>
     <collision>
-      <geometry><sphere radius="0.03"/></geometry>  <!-- Simplified collision -->
+      <geometry><sphere radius="0.03"/></geometry>
     </collision>
     <inertial>
-      <mass value="0.3"/>  <!-- Increased from 0.05 -->
+      <mass value="0.3"/>
       <origin xyz="0 0 -0.1"/>
-      <!-- Approximate as point mass: I = m*d² -->
       <inertia ixx="0.003" ixy="0" ixz="0" iyy="0.003" iyz="0" izz="0.003"/>
     </inertial>
@@ -168,5 +165,5 @@
     <axis xyz="0 1 0"/>
     <limit lower="-${M_PI/2}" upper="${M_PI/2}" effort="50" velocity="1"/>
-    <dynamics damping="0.2"/>  <!-- Added damping -->
+    <dynamics damping="0.2"/>
   </joint>
 </robot>
