Commit message: polynomial

File: catkin_ws/src/giraffe_description/urdf/giraffe.urdf.xacro (robot description, xacro)
@@ -8,8 +8,8 @@
   <xacro:property name="mic_arm_length" value="0.3" />
   <!-- Materials -->
-  <material name="gray"><color rgba="0.5 0.5 0.5 1"/></material>
+  <material name="gray"><color rgba="0 0 0 1"/></material>
   <material name="red"><color rgba="1 0 0 1"/></material>
-  <material name="green"><color rgba="0 1 0 1"/></material>
-  <material name="blue"><color rgba="0 0 1 1"/></material>
+  <material name="green"><color rgba="1 1 0 1"/></material>
+  <material name="blue"><color rgba="1 0 0 1"/></material>
   <material name="yellow"><color rgba="1 1 0 1"/></material>
   <material name="black"><color rgba="0 0 0 1"/></material>

Commit message: cleaned urdf

File: catkin_ws/src/giraffe_description/urdf/giraffe.urdf.xacro (robot description, xacro)
@@ -13,5 +13,5 @@
   <material name="light grey"><color rgba="0 0 0 0.5"/></material>
   <link name="world"/>
-  <!-- Base - Increased mass and corrected inertia -->
+  <!-- Base -->
   <link name="base_link">
     <visual>
@@ -23,7 +23,6 @@
     </collision>
     <inertial>
-      <mass value="5.0"/>  <!-- Increased from 2.0 -->
+      <mass value="5.0"/>
       <origin xyz="0 0 0"/>
-      <!-- Corrected inertia for box: I = 1/12*m*(y²+z²) -->
       <inertia ixx="0.00417" ixy="0" ixz="0" iyy="0.00417" iyz="0" izz="0.00833"/>
     </inertial>
@@ -34,5 +33,5 @@
     <origin xyz="2.5 6.0 ${ceiling_height}" rpy="0 0 0"/>
   </joint>
-  <!-- Link1: Pan - Corrected inertia for cylinder -->
+  <!-- Link1 -->
   <link name="link1">
     <visual>
@@ -57,5 +56,5 @@
     <dynamics damping="0.5"/>
   </joint>
-  <!-- Link2: Tilt - Corrected inertia and COM -->
+  <!-- Link2 -->
   <link name="link2">
     <visual>
@@ -69,7 +68,6 @@
     </collision>
     <inertial>
-      <mass value="2.0"/>  <!-- Increased from 0.7 -->
+      <mass value="2.0"/>
       <origin xyz="${arm_segment_length/2} 0 0"/>  <!-- COM at center -->
-      <!-- For cylinder along x: Ixx = 1/2*m*r², Iyy=Izz=1/12*m*(3r²+L²) -->
       <inertia ixx="0.0009" ixy="0" ixz="0" iyy="0.0417" iyz="0" izz="0.0417"/>
     </inertial>
@@ -80,8 +78,8 @@
     <origin xyz="0 0 0" rpy="0 0 0"/>
     <axis xyz="0 1 0"/>
-    <limit lower="-${2*M_PI/3}" upper="0" effort="100" velocity="1"/> <!-- Reduced range -->
-    <dynamics damping="0.5"/>  <!-- Added damping -->
+    <limit lower="-${2*M_PI/3}" upper="0" effort="100" velocity="1"/>
+    <dynamics damping="0.5"/>
   </joint>
-  <!-- Link3: Prismatic - Increased mass and corrected inertia -->
+  <!-- Link3 -->
 <link name="link3">
     <visual>
@@ -106,7 +104,7 @@
     <axis xyz="1 0 0"/>
     <limit lower="0" upper="${prismatic_max_extension}" effort="10000" velocity="0.5"/>
-    <dynamics damping="10.0" friction="2.0"/>  <!-- Increased damping -->
+    <dynamics damping="10.0" friction="2.0"/>
   </joint>
-  <!-- Link4: Microphone bar - Corrected inertia -->
+  <!-- Link4: Microphone bar -->
   <link name="link4">
     <visual>
@@ -120,7 +118,6 @@
     </collision>
     <inertial>
-      <mass value="0.5"/>  <!-- Increased from 0.1 -->
+      <mass value="0.5"/>
       <origin xyz="${mic_arm_length/2} 0 0"/>
-      <!-- For cylinder along x: Ixx = 1/2*m*r², Iyy=Izz=1/12*m*(3r²+L²) -->
       <inertia ixx="0.000025" ixy="0" ixz="0" iyy="0.00377" iyz="0" izz="0.00377"/>
     </inertial>
@@ -134,5 +131,5 @@
     <dynamics damping="0.3"/>
   </joint>
-  <!-- End-effector: microphone - Corrected inertia -->
+  <!-- End-effector: microphone -->
   <link name="ee_link">
     <visual>
